File: Current_Carrying_Pins.kicad_sch (KiCad schematic)
At the start: 0 parts

Commit message: Full schematic connection without ratio consideration.
Parts:
- added U1_1, U1_10, U1_11, U1_12, U1_13, U1_14, U1_15, U1_2, U1_3, U1_4, U1_5, U1_6, U1_7, U1_8, U1_9: ADP7104ARDZ-R7, RD_8_2_ADI, symbol Adjustable Low-Dropout Regulator:ADP7104ARDZ-R7
- added U2_1, U2_2, U2_3, U2_4, U2_5, U2_6, U2_7, U2_8: TPL0102-100PWR, PW14, symbol Digital Potentiometer:TPL0102-100PWR
- added U3_1, U3_2, U3_3, U3_4, U3_5, U3_6, U3_9: TPS259620DDAR, SOIC_20DDAR_TEX, symbol eFuse for electronic:TPS259620DDAR
Connections:
- new net: U1_10.2 (SENSE/ADJ), U2_6.3 (WA)
- new net: U1_11.2 (SENSE/ADJ), U2_6.6 (WB)
- new net: U1_1.2 (SENSE/ADJ), U2_1.3 (WA)
- new net: U1_1.8 (VIN), U1_2.8 (VIN), U3_1.5 (OUT)
- new net: U1_12.1 (VOUT), U2_7.2 (LA), U3_5.3 (EN/UVLO), U3_5.4 (IN)
- new net: U1_12.2 (SENSE/ADJ), U2_7.3 (WA)
- new net: U1_10.8 (VIN), U1_11.8 (VIN), U1_9.8 (VIN), U3_9.5 (OUT)
- new net: U1_15.1 (VOUT), U2_8.5 (LB), U3_4.3 (EN/UVLO), U3_4.4 (IN)
- new net: U1_15.2 (SENSE/ADJ), U2_8.6 (WB)
- new net: U1_7.2 (SENSE/ADJ), U2_4.3 (WA)
- new net: U1_3.8 (VIN), U1_4.8 (VIN), U1_5.8 (VIN), U1_6.8 (VIN), U1_7.8 (VIN), U1_8.8 (VIN), U3_2.5 (OUT)
- new net: U1_5.2 (SENSE/ADJ), U2_3.3 (WA)
- new net: U1_2.2 (SENSE/ADJ), U2_1.6 (WB)
- new net: U1_14.1 (VOUT), U2_8.2 (LA), U3_3.3 (EN/UVLO), U3_3.4 (IN)
- new net: U1_14.2 (SENSE/ADJ), U2_8.3 (WA)
- new net: U1_13.1 (VOUT), U2_7.5 (LB), U3_6.3 (EN/UVLO), U3_6.4 (IN)
- new net: U1_13.2 (SENSE/ADJ), U2_7.6 (WB)
- new net: U1_6.2 (SENSE/ADJ), U2_3.6 (WB)
- new net: U1_4.2 (SENSE/ADJ), U2_2.6 (WB)
- new net: U1_3.2 (SENSE/ADJ), U2_2.3 (WA)
- new net: U1_9.2 (SENSE/ADJ), U2_5.3 (WA)
- new net: U1_8.2 (SENSE/ADJ), U2_4.6 (WB)
- new net 3.3V: U2_1.14 (VDD), U2_2.14 (VDD), U2_3.14 (VDD), U2_4.14 (VDD), U2_5.14 (VDD), U2_6.14 (VDD), U2_7.14 (VDD), U2_8.14 (VDD)
- new net A0_DIGIPOT: U2_1.13 (A0), U2_2.13 (A0), U2_3.13 (A0), U2_4.13 (A0), U2_5.13 (A0), U2_6.13 (A0), U2_7.13 (A0), U2_8.13 (A0)
- new net A1_DIGIPOT: U2_1.12 (A1), U2_2.12 (A1), U2_3.12 (A1), U2_4.12 (A1), U2_5.12 (A1), U2_6.12 (A1), U2_7.12 (A1), U2_8.12 (A1)
- new net A2_DIGIPOT: U2_1.7 (A2), U2_2.7 (A2), U2_3.7 (A2), U2_4.7 (A2), U2_5.7 (A2), U2_6.7 (A2), U2_7.7 (A2), U2_8.7 (A2)
- new net Buck_Output_3.8V: U1_12.8 (VIN), U1_13.8 (VIN), U1_14.8 (VIN), U1_15.8 (VIN), U3_9.3 (EN/UVLO), U3_9.4 (IN)
- new net Enable_Pin12_2.0V_60mA: U1_1.5 (EN/UVLO)
- new net Enable_Pin13_3.6V_250mA: U1_14.5 (EN/UVLO)
- new net Enable_Pin14_3.6V_250mA: U1_15.5 (EN/UVLO)
- new net Enable_Pin19_3.6V_250mA: U1_12.5 (EN/UVLO)
- new net Enable_Pin20_2.0V_60mA: U1_2.5 (EN/UVLO)
- new net Enable_Pin27_2.6V_30mA: U1_4.5 (EN/UVLO)
- new net Enable_Pin30_2.6V_30mA: U1_5.5 (EN/UVLO)
- new net Enable_Pin32_2.6V_30mA: U1_6.5 (EN/UVLO)
- new net Enable_Pin34_2.6V_30mA: U1_7.5 (EN/UVLO)
- new net Enable_Pin39_2.6V_30mA: U1_8.5 (EN/UVLO)
- new net Enable_Pin3_2.6V_30mA: U1_3.5 (EN/UVLO)
- new net Enable_Pin41_3.0V_40mA: U1_9.5 (EN/UVLO)
- new net Enable_Pin42_3.6V_30mA: U1_13.5 (EN/UVLO)
- new net Enable_Pin6_3.0V_40mA: U1_10.5 (EN/UVLO)
- new net Enable_Pin7_3.0V_6mA: U1_11.5 (EN/UVLO)
- new net GND: U1_1.3 (GND), U1_1.6 (GND), U1_10.3 (GND), U1_10.6 (GND), U1_11.3 (GND), U1_11.6 (GND), U1_12.3 (GND), U1_12.6 (GND), U1_13.3 (GND), U1_13.6 (GND), U1_14.3 (GND), U1_14.6 (GND), U1_15.3 (GND), U1_15.6 (GND), U1_2.3 (GND), U1_2.6 (GND), U1_3.3 (GND), U1_3.6 (GND), U1_4.3 (GND), U1_4.6 (GND), U1_5.3 (GND), U1_5.6 (GND), U1_6.3 (GND), U1_6.6 (GND), U1_7.3 (GND), U1_7.6 (GND), U1_8.3 (GND), U1_8.6 (GND), U1_9.3 (GND), U1_9.6 (GND), U2_1.1 (HA), U2_1.11 (GND), U2_1.4 (HB), U2_2.1 (HA), U2_2.11 (GND), U2_2.4 (HB), U2_2.8 (VSS), U2_3.1 (HA), U2_3.11 (GND), U2_3.4 (HB), U2_3.8 (VSS), U2_4.1 (HA), U2_4.11 (GND), U2_4.4 (HB), U2_4.8 (VSS), U2_5.1 (HA), U2_5.11 (GND), U2_5.4 (HB), U2_5.8 (VSS), U2_6.1 (HA), U2_6.11 (GND), U2_6.4 (HB), U2_6.8 (VSS), U2_7.1 (HA), U2_7.11 (GND), U2_7.4 (HB), U2_7.8 (VSS), U2_8.1 (HA), U2_8.11 (GND), U2_8.4 (HB), U2_8.8 (VSS), U3_1.1 (GND), U3_2.1 (GND), U3_3.1 (GND), U3_4.1 (GND), U3_5.1 (GND), U3_6.1 (GND), U3_9.1 (GND)
- new net LDO_Fixed_3.3V: U3_1.3 (EN/UVLO), U3_1.4 (IN), U3_2.3 (EN/UVLO), U3_2.4 (IN)
- new net PG_LDO_1: U1_1.7 (PG), U1_10.7 (PG), U1_12.7 (PG), U1_14.7 (PG), U1_3.7 (PG), U1_5.7 (PG), U1_7.7 (PG), U1_9.7 (PG)
- new net PG_LDO_2: U1_11.7 (PG), U1_13.7 (PG), U1_15.7 (PG), U1_2.7 (PG), U1_4.7 (PG), U1_6.7 (PG), U1_8.7 (PG)
- new net Pin12_2.0V_60mA: U1_1.1 (VOUT), U2_1.2 (LA)
- new net Pin13_3.6V_250mA: U3_3.5 (OUT)
- new net Pin14_3.6V_250mA: U3_4.5 (OUT)
- new net Pin19_3.6V_250mA: U3_5.5 (OUT)
- new net Pin20_2.0V_60mA: U1_2.1 (VOUT), U2_1.5 (LB)
- new net Pin27_2.6V_30mA: U1_4.1 (VOUT), U2_2.5 (LB)
- new net Pin30_2.6V_30mA: U1_5.1 (VOUT), U2_3.2 (LA)
- new net Pin32_2.6V_30mA: U1_6.1 (VOUT), U2_3.5 (LB)
- new net Pin34_2.6V_30mA: U1_7.1 (VOUT), U2_4.2 (LA)
- new net Pin39_2.6V_30mA: U1_8.1 (VOUT), U2_4.5 (LB)
- new net Pin3_2.6V_30mA: U1_3.1 (VOUT), U2_2.2 (LA)
- new net Pin41_3.0V_40mA: U1_9.1 (VOUT), U2_5.2 (LA)
- new net Pin42_3.6V_30mA: U3_6.5 (OUT)
- new net Pin6_3.0V_40mA: U1_10.1 (VOUT), U2_6.2 (LA)
- new net Pin7_3.0V_6mA: U1_11.1 (VOUT), U2_6.5 (LB)
- new net SCL_Current_Carrying_Pins: U2_1.10 (SCL), U2_2.10 (SCL), U2_3.10 (SCL), U2_4.10 (SCL), U2_5.10 (SCL), U2_6.10 (SCL), U2_7.10 (SCL), U2_8.10 (SCL)
- new net SDA_Current_Carrying_Pins: U2_1.9 (SDA), U2_2.9 (SDA), U2_3.9 (SDA), U2_4.9 (SDA), U2_5.9 (SDA), U2_6.9 (SDA), U2_7.9 (SDA), U2_8.9 (SDA)
- new net VSS_DIGIPOT: U2_1.8 (VSS)
- no-connect marks 0 -> 21
Other:
- removed sheet 2.0V_Section
- removed sheet 2.6V_Section
- removed sheet 3.0V_Section
- removed sheet 3.6V-HighPower
- note removed: "I have not add connection to 3.0V section since i still have to consider where to put the extra digipot (delete if needed)"
