File: Non-Current_Carrying_Pins.kicad_sch (KiCad schematic)
At the start: 41 parts, among them U2_10 TPL0102-100PWR, U2_11 TPL0102-100PWR, U2_12 TPL0102-100PWR, U2_13 TPL0102-100PWR, U2_14 TPL0102-100PWR, U2_15 TPL0102-100PWR, U2_16 TPL0102-100PWR, U2_9 TPL0102-100PWR, U3_7 TPS259620DDAR

Commit message: Update the work from pin 1 to pin 12
Connections:
- net 3.3V: now also U2_10.14 (VDD), U2_11.14 (VDD), U2_12.14 (VDD), U2_13.14 (VDD), U2_14.14 (VDD), U2_15.14 (VDD), U2_16.14 (VDD), U2_9.14 (VDD); no longer R13.2, R14.2, R15.2, R16.2, R25.2, R26.2, R27.2, R28.2, R29.2, R30.2, R31.2, R32.2, R7.2, R8.2
- net 3.3V_eFuse: now also R13.2, R14.2, R15.2, R16.2, R25.2, R26.2, R27.2, R28.2, R29.2, R30.2, R31.2, R32.2, R7.2, R8.2; no longer U2_10.14 (VDD), U2_11.14 (VDD), U2_12.14 (VDD), U2_13.14 (VDD), U2_14.14 (VDD), U2_15.14 (VDD), U2_16.14 (VDD), U2_9.14 (VDD)
Other:
- moved on the sheet: U3_7
