File: Switchable_Pins.kicad_sch (KiCad schematic)
At the start: 41 parts, among them U2_17 TPL0102-100PWR, U2_18 TPL0102-100PWR, U2_19 TPL0102-100PWR, U2_20 TPL0102-100PWR, U2_21 TPL0102-100PWR, U2_22 TPL0102-100PWR, U2_23 TPL0102-100PWR, U2_24 TPL0102-100PWR, U3_8 TPS259620DDAR

Commit message: Update the work from pin 1 to pin 12
Connections:
- net 3.3V: now also U2_17.14 (VDD), U2_18.14 (VDD), U2_19.14 (VDD), U2_20.14 (VDD), U2_21.14 (VDD), U2_22.14 (VDD), U2_23.14 (VDD), U2_24.14 (VDD); no longer R49.2, R50.2, R51.2, R52.2, R53.2, R54.2, R55.2, R56.2, R57.2, R58.2, R59.2, R60.2, R61.2, R62.2, R63.2, R64.2
- net 3.3V_eFuse: now also R49.2, R50.2, R51.2, R52.2, R53.2, R54.2, R55.2, R56.2, R57.2, R58.2, R59.2, R60.2, R61.2, R62.2, R63.2, R64.2; no longer U2_17.14 (VDD), U2_18.14 (VDD), U2_19.14 (VDD), U2_20.14 (VDD), U2_21.14 (VDD), U2_22.14 (VDD), U2_23.14 (VDD), U2_24.14 (VDD)
Other:
- moved on the sheet: U3_8
