File: Pin1-12.kicad_sch (KiCad schematic)
At the start: 26 parts, among them U1_16 ADP7104ARDZ-R7, U1_17 ADP7104ARDZ-R7, U1_18 ADP7104ARDZ-R7, U1_19 ADP7104ARDZ-R7, U2_25 TPL0102-100PWR, U2_26 TPL0102-100PWR, U2_27 TPL0102-100PWR, U2_28 TPL0102-100PWR, U2_29 TPL0102-100PWR, U2_30 TPL0102-100PWR

Commit message: Updates on full connection for Protoboard Layout
Connections:
- net Pin4_2.0V_No_Current: now also U2_26.6 (WB); no longer U2_26.4 (HB)
- net at R71.1: now also U2_26.4 (HB); no longer U2_26.6 (WB)
Other:
- moved on the sheet: R71
Changed lines of the file:
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@@
 	(wire
 		(pts
-			(xy 294.64 144.78) (xy 251.46 144.78)
+			(xy 294.64 139.7) (xy 251.46 139.7)
 		)
 		(stroke
@@
 	(wire
 		(pts
-			(xy 251.46 139.7) (xy 330.2 139.7)
+			(xy 251.46 144.78) (xy 330.2 144.78)
 		)
 		(stroke
@@
 	(wire
 		(pts
-			(xy 302.26 144.78) (xy 303.53 144.78)
+			(xy 302.26 139.7) (xy 303.53 139.7)
 		)
 		(stroke
@@
 	(global_label "3.3V_eFuse"
 		(shape input)
-		(at 303.53 144.78 0)
+		(at 303.53 139.7 0)
 		(fields_autoplaced yes)
 		(effects
@@
 		)
 		(property "Intersheetrefs" "${INTERSHEET_REFS}"
-			(at 310.6276 144.78 0)
+			(at 310.6276 139.7 0)
 			(hide yes)
 			(show_name no)
@@
 	(global_label "Pin4_2.0V_No_Current"
 		(shape output)
-		(at 330.2 139.7 0)
+		(at 330.2 144.78 0)
 		(fields_autoplaced yes)
 		(effects
@@
 		)
 		(property "Intersheetrefs" "${INTERSHEET_REFS}"
-			(at 353.8679 139.7 0)
+			(at 353.8679 144.78 0)
 			(hide yes)
 			(show_name no)
@@
 	(symbol
 		(lib_id "Device:R")
-		(at 298.45 144.78 90)
+		(at 298.45 139.7 90)
 		(mirror x)
 		(unit 1)
@@
 		(in_pos_files yes)
 		(dnp no)
-		(fields_autoplaced yes)
 		(property "Reference" "R71"
-			(at 298.45 151.13 90)
+			(at 298.45 146.05 90)
 			(show_name no)
 			(do_not_autoplace no)
@@
 		)
 		(property "Value" "R"
-			(at 298.45 148.59 90)
+			(at 298.45 143.51 90)
 			(show_name no)
 			(do_not_autoplace no)
@@
 		)
 		(property "Footprint" ""
-			(at 298.45 143.002 90)
+			(at 298.45 137.922 90)
 			(hide yes)
 			(show_name no)
@@
 		)
 		(property "Datasheet" ""
-			(at 298.45 144.78 0)
+			(at 298.45 139.7 0)
 			(hide yes)
 			(show_name no)
@@
 		)
 		(property "Description" "Resistor"
-			(at 298.45 144.78 0)
+			(at 298.45 139.7 0)
 			(hide yes)
 			(show_name no)
@@
 		(in_pos_files yes)
 		(dnp no)
-		(fields_autoplaced yes)
 		(property "Reference" "R69"
 			(at 283.21 148.59 90)
@@
 		(lib_id "power:GND")
 		(at 287.02 142.24 90)
-		(mirror x)
 		(unit 1)
 		(body_style 1)
@@
 		)
 		(property "Value" "GND"
-			(at 290.83 142.2401 90)
+			(at 290.83 142.2399 90)
 			(show_name no)
 			(do_not_autoplace no)

Commit message: Update on Anotation for each components
Parts:
- renumbered R67 to R1, R73 to R10, R79 to R11, R74 to R12, R80 to R13, R76 to R14, R81 to R15, R77 to R16, R65 to R2, R68 to R3, R66 to R4, R71 to R5, R69 to R6, R70 to R7, R72 to R8, R75 to R9, U1_16 to U1_1, U1_17 to U1_2, U1_18 to U1_3, U1_19 to U1_4, U2_25 to U2_1, U2_26 to U2_2, U2_27 to U2_3, U2_28 to U2_4, U2_29 to U2_5, U2_30 to U2_6
