File: Pin13-23.kicad_sch (KiCad schematic)
At the start: 5 parts, among them U1_20 ADP7104ARDZ-R7, U1_21 ADP7104ARDZ-R7, U2_31 TPL0102-100PWR, U3_14 TPS259620DDAR, U3_15 TPS259620DDAR

Commit message: Updates on full connection for Protoboard Layout
Parts:
- added R78, R82, R83, R84, R85, R86, R87, R88, R89, R90, R91, R92, R93, R95: R, symbol Device:R
- added U1_22, U1_23: ADP7104ARDZ-R7, RD_8_2_ADI, symbol Adjustable Low-Dropout Regulator:ADP7104ARDZ-R7
- added U2_32, U2_33, U2_34, U2_35, U2_36: TPL0102-100PWR, PW14, symbol Digital Potentiometer:TPL0102-100PWR
- added U3_16: TPS259620DDAR, SOIC_20DDAR_TEX, symbol eFuse for electronic:TPS259620DDAR
Connections:
- net 3.3V is gone; now on net GND: U2_31.14 (VDD)
- net A0_DIGIPOT is gone; now on net GND: U2_31.13 (A0)
- net A1_DIGIPOT is gone; now on net GND: U2_31.12 (A1)
- net A2_DIGIPOT is gone; now on net GND: U2_31.7 (A2)
- net Buck_Output_3.8V: now also U1_23.8 (VIN)
- net GND: now also R78.2, R82.2, R83.2, R87.2, R89.2, R90.2, R93.2, U1_22.3 (GND), U1_22.6 (GND), U1_23.3 (GND), U1_23.6 (GND), U2_32.11 (GND), U2_32.12 (A1), U2_32.13 (A0), U2_32.14 (VDD), U2_32.7 (A2), U2_32.8 (VSS), U2_33.11 (GND), U2_33.12 (A1), U2_33.13 (A0), U2_33.14 (VDD), U2_33.7 (A2), U2_33.8 (VSS), U2_34.1 (HA), U2_34.11 (GND), U2_34.12 (A1), U2_34.13 (A0), U2_34.14 (VDD), U2_34.4 (HB), U2_34.7 (A2), U2_34.8 (VSS), U2_35.11 (GND), U2_35.12 (A1), U2_35.13 (A0), U2_35.14 (VDD), U2_35.7 (A2), U2_35.8 (VSS), U2_36.11 (GND), U2_36.12 (A1), U2_36.13 (A0), U2_36.14 (VDD), U2_36.7 (A2), U2_36.8 (VSS), U3_16.1 (GND)
- net PG_LDO_1: now also U1_23.7 (PG)
- net PG_LDO_2: now also U1_22.7 (PG)
- net SCL_Current_Carrying_Pins renamed SCL_Pin13to23
- net SCL_Pin13to23: now also U2_32.10 (SCL), U2_33.10 (SCL), U2_34.10 (SCL), U2_35.10 (SCL), U2_36.10 (SCL)
- net SDA_Current_Carrying_Pins renamed SDA_Pin13to23
- net SDA_Pin13to23: now also U2_32.9 (SDA), U2_33.9 (SDA), U2_34.9 (SDA), U2_35.9 (SDA), U2_36.9 (SDA)
- new net: R88.1, U2_32.4 (HB)
- new net: U1_22.2 (SENSE/ADJ), U2_34.6 (WB)
- new net: R78.1, U2_33.2 (LA)
- new net: R92.1, U2_35.1 (HA)
- new net: R90.1, U2_35.2 (LA)
- new net: R91.1, U2_35.4 (HB)
- new net: R89.1, U2_35.5 (LB)
- new net: U1_23.1 (VOUT), U2_34.2 (LA), U3_16.3 (EN/UVLO), U3_16.4 (IN)
- new net: U1_23.2 (SENSE/ADJ), U2_34.3 (WA)
- new net: R82.1, U2_32.2 (LA)
- new net: R83.1, U2_33.5 (LB)
- new net: R95.1, U2_36.1 (HA)
- new net: R84.1, U2_32.1 (HA)
- new net: R93.1, U2_36.2 (LA)
- new net: R86.1, U2_33.4 (HB)
- new net: R85.1, U2_33.1 (HA)
- new net: R87.1, U2_32.5 (LB)
- new net 3.3V_eFuse: R84.2, R85.2, R86.2, R88.2, R91.2, R92.2, R95.2
- new net Enable_Pin19_3.6V_250mA: U1_23.5 (EN/UVLO)
- new net Enable_Pin20_2.0V_60mA: U1_22.5 (EN/UVLO)
- new net Pin15_1.2V_No_Current: U2_32.3 (WA)
- new net Pin16_Either0Vor2V_No_Current: U2_32.6 (WB)
- new net Pin17_Either0Vor2V_No_Current: U2_33.3 (WA)
- new net Pin18_1.2V_No_Current: U2_33.6 (WB)
- new net Pin19_3.6V_250mA: U3_16.5 (OUT)
- new net Pin20_2.0V_60mA: U1_22.1 (VOUT), U2_34.5 (LB)
- new net Pin21_1.2V_No_Current: U2_35.3 (WA)
- new net Pin22_Either0Vor2V_No_Current: U2_35.6 (WB)
- new net Pin23_2.0V_No_Current: U2_36.3 (WA)
- new net eFuse_2.0V_pins: U1_22.8 (VIN)
- no-connect marks 4 -> 7
Other:
- moved on the sheet: U1_20, U1_21, U2_31, U3_14, U3_15

Commit message: Update on Anotation for each components
Parts:
- renumbered R84 to R17, R82 to R18, R88 to R19, R87 to R20, R85 to R21, R78 to R22, R86 to R23, R83 to R24, R92 to R25, R90 to R26, R91 to R27, R89 to R28, R95 to R29, R93 to R30, U1_20 to U1_5, U1_21 to U1_6, U1_23 to U1_7, U1_22 to U1_8, U2_34 to U2_10, U2_35 to U2_11, U2_36 to U2_12, U2_31 to U2_7, U2_32 to U2_8, U2_33 to U2_9, U3_14 to U3_5, U3_15 to U3_6, U3_16 to U3_7
