File: Pin24-35.kicad_sch (KiCad schematic)
At the start: 0 parts

Commit message: Updates on full connection for Protoboard Layout
Parts:
- added R100, R101, R102, R103, R104, R105, R106, R107, R108, R109, R110, R94, R96, R97, R98, R99: R, symbol Device:R
- added U1_24, U1_25, U1_26, U1_27: ADP7104ARDZ-R7, RD_8_2_ADI, symbol Adjustable Low-Dropout Regulator:ADP7104ARDZ-R7
- added U2_37, U2_38, U2_39, U2_40, U2_41, U2_42: TPL0102-100PWR, PW14, symbol Digital Potentiometer:TPL0102-100PWR
Connections:
- new net: R110.1, U2_42.4 (HB)
- new net: R97.1, U2_38.2 (LA)
- new net: U1_27.2 (SENSE/ADJ), U2_42.3 (WA)
- new net: R109.1, U2_42.5 (LB)
- new net: R96.1, U2_37.2 (LA)
- new net: U1_26.2 (SENSE/ADJ), U2_41.3 (WA)
- new net: R108.1, U2_41.4 (HB)
- new net: R107.1, U2_41.5 (LB)
- new net: R99.1, U2_37.4 (HB)
- new net: U1_25.2 (SENSE/ADJ), U2_40.3 (WA)
- new net: R106.1, U2_40.4 (HB)
- new net: R105.1, U2_40.5 (LB)
- new net: R101.1, U2_39.2 (LA)
- new net: R98.1, U2_37.1 (HA)
- new net: R94.1, U2_37.5 (LB)
- new net: U1_24.2 (SENSE/ADJ), U2_38.6 (WB)
- new net: R104.1, U2_39.4 (HB)
- new net: R102.1, U2_39.5 (LB)
- new net: R103.1, U2_39.1 (HA)
- new net: R100.1, U2_38.1 (HA)
- new net 3.3V: U2_37.14 (VDD), U2_38.13 (A0), U2_38.14 (VDD), U2_39.12 (A1), U2_39.14 (VDD), U2_40.12 (A1), U2_40.13 (A0), U2_40.14 (VDD), U2_41.14 (VDD), U2_41.7 (A2), U2_42.13 (A0), U2_42.14 (VDD), U2_42.7 (A2)
- new net 3.3V_eFuse: R100.2, R103.2, R104.2, R106.2, R108.2, R110.2, R98.2, R99.2
- new net Enable_Pin27_2.6V_30mA: U1_24.5 (EN/UVLO)
- new net Enable_Pin30_2.6V_30mA: U1_25.5 (EN/UVLO)
- new net Enable_Pin32_2.6V_30mA: U1_26.5 (EN/UVLO)
- new net Enable_Pin34_2.6V_30mA: U1_27.5 (EN/UVLO)
- new net GND: R101.2, R102.2, R105.2, R107.2, R109.2, R94.2, R96.2, R97.2, U1_24.3 (GND), U1_24.6 (GND), U1_25.3 (GND), U1_25.6 (GND), U1_26.3 (GND), U1_26.6 (GND), U1_27.3 (GND), U1_27.6 (GND), U2_37.11 (GND), U2_37.12 (A1), U2_37.13 (A0), U2_37.7 (A2), U2_37.8 (VSS), U2_38.11 (GND), U2_38.12 (A1), U2_38.4 (HB), U2_38.7 (A2), U2_38.8 (VSS), U2_39.11 (GND), U2_39.13 (A0), U2_39.7 (A2), U2_39.8 (VSS), U2_40.1 (HA), U2_40.11 (GND), U2_40.7 (A2), U2_40.8 (VSS), U2_41.1 (HA), U2_41.11 (GND), U2_41.12 (A1), U2_41.13 (A0), U2_41.8 (VSS), U2_42.1 (HA), U2_42.11 (GND), U2_42.12 (A1), U2_42.8 (VSS)
- new net PG_LDO_1: U1_25.7 (PG), U1_26.7 (PG), U1_27.7 (PG)
- new net PG_LDO_2: U1_24.7 (PG)
- new net Pin24_2.0V_No_Current: U2_37.3 (WA)
- new net Pin25_Either0Vor2V_No_Current: U2_37.6 (WB)
- new net Pin26_Either0Vor2V_No_Current: U2_38.3 (WA)
- new net Pin27_2.6V_30mA: U1_24.1 (VOUT), U2_38.5 (LB)
- new net Pin28_1.0V_No_Current: U2_39.3 (WA)
- new net Pin29_1.0V_No_Current: U2_39.6 (WB)
- new net Pin30_2.6V_30mA: U1_25.1 (VOUT), U2_40.2 (LA)
- new net Pin31_1.0V_No_Current: U2_40.6 (WB)
- new net Pin32_2.6V_30mA: U1_26.1 (VOUT), U2_41.2 (LA)
- new net Pin33_1.0V_No_Current: U2_41.6 (WB)
- new net Pin34_2.6V_30mA: U1_27.1 (VOUT), U2_42.2 (LA)
- new net Pin35_1.2V_No_Current: U2_42.6 (WB)
- new net SCL_Pin24to35: U2_37.10 (SCL), U2_38.10 (SCL), U2_39.10 (SCL), U2_40.10 (SCL), U2_41.10 (SCL), U2_42.10 (SCL)
- new net SDA_Pin24to35: U2_37.9 (SDA), U2_38.9 (SDA), U2_39.9 (SDA), U2_40.9 (SDA), U2_41.9 (SDA), U2_42.9 (SDA)
- new net eFuse_2.6V_pins: U1_24.8 (VIN), U1_25.8 (VIN), U1_26.8 (VIN), U1_27.8 (VIN)
- no-connect marks 0 -> 4
Other:
- note added: "A0_DIGIPOT"
- note added: "A1_DIGIPOT"
- note added: "A2_DIGIPOT"

Commit message: Update on Anotation for each components
Parts:
- renumbered R98 to R31, R96 to R32, R99 to R33, R94 to R34, R100 to R35, R97 to R36, R103 to R37, R101 to R38, R104 to R39, R102 to R40, R106 to R41, R105 to R42, R108 to R43, R107 to R44, R110 to R45, R109 to R46, U1_25 to U1_10, U1_26 to U1_11, U1_27 to U1_12, U1_24 to U1_9, U2_37 to U2_13, U2_38 to U2_14, U2_39 to U2_15, U2_40 to U2_16, U2_41 to U2_17, U2_42 to U2_18
