File: Pin36-46.kicad_sch (KiCad schematic)
At the start: 0 parts

Commit message: Updates on full connection for Protoboard Layout
Parts:
- added R111, R112, R113, R114, R115, R116, R117, R118, R119, R120, R121, R122, R125, R126: R, symbol Device:R
- added U1_28, U1_29, U1_30: ADP7104ARDZ-R7, RD_8_2_ADI, symbol Adjustable Low-Dropout Regulator:ADP7104ARDZ-R7
- added U2_43, U2_44, U2_45, U2_46, U2_47: TPL0102-100PWR, PW14, symbol Digital Potentiometer:TPL0102-100PWR
- added U3_17: TPS259620DDAR, SOIC_20DDAR_TEX, symbol eFuse for electronic:TPS259620DDAR
Connections:
- new net: R125.1, U2_47.1 (HA)
- new net: R122.1, U2_47.5 (LB)
- new net: R113.1, U2_43.1 (HA)
- new net: R111.1, U2_43.2 (LA)
- new net: R114.1, U2_43.4 (HB)
- new net: R112.1, U2_43.5 (LB)
- new net: U1_30.1 (VOUT), U2_45.5 (LB), U3_17.3 (EN/UVLO), U3_17.4 (IN)
- new net: U1_28.2 (SENSE/ADJ), U2_44.3 (WA)
- new net: U1_30.2 (SENSE/ADJ), U2_45.6 (WB)
- new net: R121.1, U2_47.2 (LA)
- new net: R116.1, U2_44.4 (HB)
- new net: R120.1, U2_46.4 (HB)
- new net: R126.1, U2_47.4 (HB)
- new net: R117.1, U2_46.2 (LA)
- new net: R115.1, U2_44.5 (LB)
- new net: R119.1, U2_46.1 (HA)
- new net: R118.1, U2_46.5 (LB)
- new net: U1_29.2 (SENSE/ADJ), U2_45.3 (WA)
- new net 3.3V: U2_43.14 (VDD), U2_44.13 (A0), U2_44.14 (VDD), U2_45.12 (A1), U2_45.14 (VDD), U2_46.12 (A1), U2_46.13 (A0), U2_46.14 (VDD), U2_47.14 (VDD), U2_47.7 (A2)
- new net 3.3V_eFuse: R113.2, R114.2, R116.2, R119.2, R120.2, R125.2, R126.2
- new net Buck_Output_3.8V: U1_30.8 (VIN)
- new net Enable_Pin39_2.6V_30mA: U1_28.5 (EN/UVLO)
- new net Enable_Pin41_3.0V_40mA: U1_29.5 (EN/UVLO)
- new net Enable_Pin42_3.6V_30mA: U1_30.5 (EN/UVLO)
- new net GND: R111.2, R112.2, R115.2, R117.2, R118.2, R121.2, R122.2, U1_28.3 (GND), U1_28.6 (GND), U1_29.3 (GND), U1_29.6 (GND), U1_30.3 (GND), U1_30.6 (GND), U2_43.11 (GND), U2_43.12 (A1), U2_43.13 (A0), U2_43.7 (A2), U2_43.8 (VSS), U2_44.1 (HA), U2_44.11 (GND), U2_44.12 (A1), U2_44.7 (A2), U2_44.8 (VSS), U2_45.1 (HA), U2_45.11 (GND), U2_45.13 (A0), U2_45.4 (HB), U2_45.7 (A2), U2_45.8 (VSS), U2_46.11 (GND), U2_46.7 (A2), U2_46.8 (VSS), U2_47.11 (GND), U2_47.12 (A1), U2_47.13 (A0), U2_47.8 (VSS), U3_17.1 (GND)
- new net PG_LDO_1: U1_28.7 (PG), U1_29.7 (PG)
- new net PG_LDO_2: U1_30.7 (PG)
- new net Pin37_Either0Vor2V_No_Current: U2_43.3 (WA)
- new net Pin38_Either0Vor2V_No_Current: U2_43.6 (WB)
- new net Pin39_2.6V_30mA: U1_28.1 (VOUT), U2_44.2 (LA)
- new net Pin40_2.0V_No_Current: U2_44.6 (WB)
- new net Pin41_3.0V_40mA: U1_29.1 (VOUT), U2_45.2 (LA)
- new net Pin42_3.6V_30mA: U3_17.5 (OUT)
- new net Pin43_1.2V_No_Current: U2_46.3 (WA)
- new net Pin44_Either0Vor2V_No_Current: U2_46.6 (WB)
- new net Pin45_Either0Vor2V_No_Current: U2_47.3 (WA)
- new net Pin46_Either0Vor2V_No_Current: U2_47.6 (WB)
- new net SCL_Pin36to46: U2_43.10 (SCL), U2_44.10 (SCL), U2_45.10 (SCL), U2_46.10 (SCL), U2_47.10 (SCL)
- new net SDA_Pin36to46: U2_43.9 (SDA), U2_44.9 (SDA), U2_45.9 (SDA), U2_46.9 (SDA), U2_47.9 (SDA)
- new net eFuse_2.6V_pins: U1_28.8 (VIN)
- new net eFuse_3.0V_pins: U1_29.8 (VIN)
- no-connect marks 0 -> 4
Other:
- note added: "A0_DIGIPOT"
- note added: "A1_DIGIPOT"
- note added: "A2_DIGIPOT"

Commit message: Update on Anotation for each components
Parts:
- renumbered R113 to R47, R111 to R48, R114 to R49, R112 to R50, R116 to R51, R115 to R52, R119 to R53, R117 to R54, R120 to R55, R118 to R56, R125 to R57, R121 to R58, R126 to R59, R122 to R60, U1_28 to U1_13, U1_29 to U1_14, U1_30 to U1_15, U2_43 to U2_19, U2_44 to U2_20, U2_45 to U2_21, U2_46 to U2_22, U2_47 to U2_23, U3_17 to U3_8
