File: Smart_DC_PowerSupply.kicad_sch (KiCad schematic)
At the start: 7 parts, among them J1 USB_C_Receptacle_PowerOnly_24P, U0_1 TPS62A03DRLR, U4_1 MC74HC595ADTR2G, U4_2 MC74HC595ADTR2G, U5_1 ADP7105ARDZ-3.3-R7, U5_2 ADP150AUJZ-3.3-R7, U6_1 PCA9546APW_118

Commit message: Update the work from pin 1 to pin 12
Parts:
- added U3_10, U3_11, U3_12, U3_13: TPS259620DDAR, SOIC_20DDAR_TEX, symbol eFuse for electronic:TPS259620DDAR
Connections:
- net 3.3V: now also U3_13.3 (EN/UVLO), U3_13.4 (IN)
- net Buck_Output_3.8V: now also U3_10.3 (EN/UVLO), U3_10.4 (IN), U3_11.3 (EN/UVLO), U3_11.4 (IN), U3_12.3 (EN/UVLO), U3_12.4 (IN)
- net GND: now also U3_10.1 (GND), U3_11.1 (GND), U3_12.1 (GND), U3_13.1 (GND)
- new net 3.3V_eFuse: U3_13.5 (OUT)
- new net eFuse_2.0V_pins: U3_12.5 (OUT)
- new net eFuse_2.6V_pins: U3_11.5 (OUT)
- new net eFuse_3.0V_pins: U3_10.5 (OUT)
- no-connect marks 8 -> 12
Other:
- added sheet Pin1-12 (Pin1-12.kicad_sch)
- added sheet Pin13-23 (Pin13-23.kicad_sch)
- added sheet Pin24-35 (Pin24-35.kicad_sch)
- added sheet Pin36-46 (Pin36-46.kicad_sch)
- note removed: "3.8V"
- moved on the sheet: J1, U0_1, U4_1, U4_2, U5_1, U5_2, U6_1

Commit message: Updates on full connection for Protoboard Layout
Connections:
- net SCL_Pin36to46: now reaches U6_1.11 (SD3)
- net SDA_Pin36to46: now reaches U6_1.12 (SC3)
- net SCL_Current_Carrying_Pins renamed SCL_Pin1to12
- net SCL_Non_Current_Carrying_Pins renamed SCL_Pin13to23
- net SCL_Switchable_Pins renamed SCL_Pin24to35
- net SDA_Current_Carrying_Pins renamed SDA_Pin1to12
- net SDA_Non_Current_Carrying_Pins renamed SDA_Pin13to23
- net SDA_Switchable_Pins renamed SDA_Pin24to35
- no-connect marks 12 -> 10
Other:
- removed sheet Current_Carrying_Pins
- removed sheet Non-Current_Carrying_Pins
- removed sheet Switchable_Pins
- moved on the sheet: U4_1, U4_2, U6_1

Commit message: Update on Anotation for each components
Parts:
- renumbered U3_10 to U3_1, U3_11 to U3_2, U3_12 to U3_3, U3_13 to U3_4
Changed lines of the file:
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@@
 		(dnp no)
 		(fields_autoplaced yes)
-		(property "Reference" "#PWR0131"
+		(property "Reference" "#PWR014"
 			(at 143.51 354.33 0)
 			(hide yes)
@@
 			(project "Smart_DC_PowerSupply"
 				(path "/eed9697a-d7f2-404b-b4ca-1333beb8d3f8"
-					(reference "#PWR0131")
+					(reference "#PWR014")
 					(unit 1)
 				)
@@
 		(dnp no)
 		(fields_autoplaced yes)
-		(property "Reference" "#PWR0162"
+		(property "Reference" "#PWR04"
 			(at 214.63 81.28 0)
 			(hide yes)
@@
 			(project "Smart_DC_PowerSupply"
 				(path "/eed9697a-d7f2-404b-b4ca-1333beb8d3f8"
-					(reference "#PWR0162")
+					(reference "#PWR04")
 					(unit 1)
 				)
@@
 		(dnp no)
 		(fields_autoplaced yes)
-		(property "Reference" "#PWR021"
+		(property "Reference" "#PWR012"
 			(at 85.09 311.15 0)
 			(hide yes)
@@
 			(project "Smart_DC_PowerSupply"
 				(path "/eed9697a-d7f2-404b-b4ca-1333beb8d3f8"
-					(reference "#PWR021")
+					(reference "#PWR012")
 					(unit 1)
 				)
@@
 		(dnp no)
 		(fields_autoplaced yes)
-		(property "Reference" "U3_10"
+		(property "Reference" "U3_1"
 			(at 246.38 20.32 0)
 			(show_name no)
@@
 			(project "Smart_DC_PowerSupply"
 				(path "/eed9697a-d7f2-404b-b4ca-1333beb8d3f8"
-					(reference "U3_10")
+					(reference "U3_1")
 					(unit 1)
 				)
@@
 		(dnp no)
 		(fields_autoplaced yes)
-		(property "Reference" "#PWR05"
+		(property "Reference" "#PWR06"
 			(at 289.56 187.96 0)
 			(hide yes)
@@
 			(project "Smart_DC_PowerSupply"
 				(path "/eed9697a-d7f2-404b-b4ca-1333beb8d3f8"
-					(reference "#PWR05")
+					(reference "#PWR06")
 					(unit 1)
 				)
@@
 		(in_pos_files yes)
 		(dnp no)
-		(property "Reference" "#PWR0132"
+		(property "Reference" "#PWR016"
 			(at 85.09 361.95 0)
 			(hide yes)
@@
 			(project "Smart_DC_PowerSupply"
 				(path "/eed9697a-d7f2-404b-b4ca-1333beb8d3f8"
-					(reference "#PWR0132")
+					(reference "#PWR016")
 					(unit 1)
 				)
@@
 		(dnp no)
 		(fields_autoplaced yes)
-		(property "Reference" "#PWR0129"
+		(property "Reference" "#PWR017"
 			(at 143.51 372.11 0)
 			(hide yes)
@@
 			(project "Smart_DC_PowerSupply"
 				(path "/eed9697a-d7f2-404b-b4ca-1333beb8d3f8"
-					(reference "#PWR0129")
+					(reference "#PWR017")
 					(unit 1)
 				)
@@
 		(dnp no)
 		(fields_autoplaced yes)
-		(property "Reference" "U3_11"
+		(property "Reference" "U3_2"
 			(at 246.38 71.12 0)
 			(show_name no)
@@
 			(project "Smart_DC_PowerSupply"
 				(path "/eed9697a-d7f2-404b-b4ca-1333beb8d3f8"
-					(reference "U3_11")
+					(reference "U3_2")
 					(unit 1)
 				)
@@
 		(dnp no)
 		(fields_autoplaced yes)
-		(property "Reference" "U3_12"
+		(property "Reference" "U3_3"
 			(at 246.38 121.92 0)
 			(show_name no)
@@
 			(project "Smart_DC_PowerSupply"
 				(path "/eed9697a-d7f2-404b-b4ca-1333beb8d3f8"
-					(reference "U3_12")
+					(reference "U3_3")
 					(unit 1)
 				)
@@
 		(dnp no)
 		(fields_autoplaced yes)
-		(property "Reference" "#PWR022"
+		(property "Reference" "#PWR011"
 			(at 149.86 285.75 0)
 			(hide yes)
@@
 			(project "Smart_DC_PowerSupply"
 				(path "/eed9697a-d7f2-404b-b4ca-1333beb8d3f8"
-					(reference "#PWR022")
+					(reference "#PWR011")
 					(unit 1)
 				)
@@
 		(dnp no)
 		(fields_autoplaced yes)
-		(property "Reference" "#PWR03"
+		(property "Reference" "#PWR07"
 			(at 212.09 190.5 0)
 			(hide yes)
@@
 			(project "Smart_DC_PowerSupply"
 				(path "/eed9697a-d7f2-404b-b4ca-1333beb8d3f8"
-					(reference "#PWR03")
+					(reference "#PWR07")
 					(unit 1)
 				)
@@
 		(dnp no)
 		(fields_autoplaced yes)
-		(property "Reference" "#PWR023"
+		(property "Reference" "#PWR013"
 			(at 149.86 330.2 0)
 			(hide yes)
@@
 			(project "Smart_DC_PowerSupply"
 				(path "/eed9697a-d7f2-404b-b4ca-1333beb8d3f8"
-					(reference "#PWR023")
+					(reference "#PWR013")
 					(unit 1)
 				)
@@
 		(dnp no)
 		(fields_autoplaced yes)
-		(property "Reference" "#PWR0163"
+		(property "Reference" "#PWR05"
 			(at 214.63 132.08 0)
 			(hide yes)
@@
 			(project "Smart_DC_PowerSupply"
 				(path "/eed9697a-d7f2-404b-b4ca-1333beb8d3f8"
-					(reference "#PWR0163")
+					(reference "#PWR05")
 					(unit 1)
 				)
@@
 		(dnp no)
 		(fields_autoplaced yes)
-		(property "Reference" "#PWR04"
+		(property "Reference" "#PWR08"
 			(at 212.09 236.22 0)
 			(hide yes)
@@
 			(project "Smart_DC_PowerSupply"
 				(path "/eed9697a-d7f2-404b-b4ca-1333beb8d3f8"
-					(reference "#PWR04")
+					(reference "#PWR08")
 					(unit 1)
 				)
@@
 		(dnp no)
 		(fields_autoplaced yes)
-		(property "Reference" "#PWR020"
+		(property "Reference" "#PWR010"
 			(at 85.09 266.7 0)
 			(hide yes)
@@
 			(project "Smart_DC_PowerSupply"
 				(path "/eed9697a-d7f2-404b-b4ca-1333beb8d3f8"
-					(reference "#PWR020")
+					(reference "#PWR010")
 					(unit 1)
 				)
@@
 		(dnp no)
 		(fields_autoplaced yes)
-		(property "Reference" "#PWR0161"
+		(property "Reference" "#PWR01"
 			(at 214.63 30.48 0)
 			(hide yes)
@@
 			(project "Smart_DC_PowerSupply"
 				(path "/eed9697a-d7f2-404b-b4ca-1333beb8d3f8"
-					(reference "#PWR0161")
+					(reference "#PWR01")
 					(unit 1)
 				)
@@
 		(dnp no)
 		(fields_autoplaced yes)
-		(property "Reference" "#PWR0164"
+		(property "Reference" "#PWR09"
 			(at 298.45 259.08 0)
 			(hide yes)
@@
 			(project "Smart_DC_PowerSupply"
 				(path "/eed9697a-d7f2-404b-b4ca-1333beb8d3f8"
-					(reference "#PWR0164")
+					(reference "#PWR09")
 					(unit 1)
 				)
@@
 		(dnp no)
 		(fields_autoplaced yes)
-		(property "Reference" "#PWR0130"
+		(property "Reference" "#PWR015"
 			(at 143.51 356.87 0)
 			(hide yes)
@@
 			(project "Smart_DC_PowerSupply"
 				(path "/eed9697a-d7f2-404b-b4ca-1333beb8d3f8"
-					(reference "#PWR0130")
+					(reference "#PWR015")
 					(unit 1)
 				)
@@
 		(dnp no)
 		(fields_autoplaced yes)
-		(property "Reference" "U3_13"
+		(property "Reference" "U3_4"
 			(at 334.01 248.92 0)
 			(show_name no)
@@
 			(project "Smart_DC_PowerSupply"
 				(path "/eed9697a-d7f2-404b-b4ca-1333beb8d3f8"
-					(reference "U3_13")
+					(reference "U3_4")
 					(unit 1)
 				)
@@
 		(dnp no)
 		(fields_autoplaced yes)
-		(property "Reference" "#PWR01"
+		(property "Reference" "#PWR03"
 			(at 63.5 86.36 0)
 			(hide yes)
@@
 			(project "Smart_DC_PowerSupply"
 				(path "/eed9697a-d7f2-404b-b4ca-1333beb8d3f8"
-					(reference "#PWR01")
-					(unit 1)
-				)
+					(reference "#PWR03")
+					(unit 1)
+				)
